File: BBPower/BBPower.kicad_pcb (KiCad board)
At the start: 2 copper layers, 22 parts, among them J1 USB_C_Receptacle, J2 Conn_01x04, J3 Conn_01x04, J4 Conn_01x04, J5 Conn_01x04, J6 Screw_Terminal_01x02, SW1 SW_DIP_x03, SW2 OS103012MU2QP1, SW3 OS103012MU2QP1, U1 CH224K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

Commit message: psb layout
Parts:
- moved SW3 65.4 mm to (149.5, 96.4), turned to -90 degrees
- moved J5 63.5 mm to (150.8, 108.0)
- moved J4 61.8 mm to (148.3, 108.0)
- moved R7 56.4 mm to (136.8, 75.8), turned to 90 degrees
- moved J6 55.9 mm to (114.0, 95.9)
- moved R8 55.7 mm to (139.4, 75.8), turned to 90 degrees
- moved R9 55.7 mm to (141.8, 75.8), turned to 90 degrees
- moved SW1 55.4 mm to (126.7, 93.8), turned to 90 degrees
- moved C1 51.5 mm to (128.0, 75.9), turned to -90 degrees
- moved R1 47.6 mm to (122.9, 75.8), turned to -90 degrees
- moved R2 44.4 mm to (125.4, 75.8), turned to 90 degrees
- moved SW2 42.4 mm to (103.8, 96.4), turned to -90 degrees
- moved J2 39.1 mm to (102.6, 108.0)
- moved J3 38.8 mm to (105.1, 108.0)
- moved R6 35.2 mm to (104.5, 77.1), turned to -90 degrees
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Connections:
- J1 pad B6: DP -> unconnected-(J1-D+-PadB6)
- J1 pad B7: DM -> unconnected-(J1-D--PadB7)
Routing:
- net VBUS: track 0.00 -> 95.7 mm, vias 0 -> 3
- net +3V3: track 0.00 -> 78.1 mm
- net +5V: track 0.00 -> 72.4 mm, vias 0 -> 1
- net CFG1: track 0.00 -> 47.6 mm
- net CFG3: track 0.00 -> 37.5 mm
- net CFG2: track 0.00 -> 35.3 mm
- net Net-(U1-VBUS): track 0.00 -> 30.9 mm, vias 0 -> 2
- net VDD: track 0.00 -> 30.5 mm, vias 0 -> 4
- net CC2: track 0.00 -> 26.4 mm, vias 0 -> 2
- net Net-(J4-Pin_1): track 0.00 -> 26.2 mm
- net CC1: track 0.00 -> 23.9 mm, vias 0 -> 2
- net GND: track 0.00 -> 21.5 mm, vias 0 -> 7
- net Net-(J2-Pin_1): track 0.00 -> 17.4 mm
- net DM: track 0.00 -> 12.6 mm, vias 0 -> 2
- net DP: track 0.00 -> 11.9 mm, vias 0 -> 2
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- added copper zone on In1.Cu, net GND
Other:
- board outline added: 52.7 x 55.9 mm
- copper layers 2 -> 4
- board text added: "BREADBOARD BUDDY REV.0 A. LEVINE"
- board text added: "JLCJLCJLC"

Commit message: pcb updates & production file
Parts:
- SW1: footprint Button_Switch_SMD:SW_DIP_SPSTx03_Slide_9.78x9.8mm_W8.61mm_P2.54mm -> Library:SW_DS04-254-1L-03BK
- moved J6 4.45 mm to (114.0, 91.4)
- moved SW1 2.42 mm to (127.0, 91.4)
- moved R4 0.95 mm to (113.0, 77.1)
- moved R5 0.95 mm to (106.0, 77.1)
- moved R6 0.95 mm to (103.5, 77.1)
- moved U3 0.95 mm to (106.0, 69.8)
- moved R3 0.95 mm to (115.6, 77.1)
- moved U2 0.95 mm to (115.6, 69.8)
Routing:
- net VBUS: track 95.7 -> 115.9 mm
- net GND: track 21.5 -> 12.1 mm, vias 7 -> 6
- net CFG1: track 47.6 -> 44.8 mm
- net +5V: track 72.4 -> 69.8 mm
- net +3V3: track 78.1 -> 75.5 mm
- net CFG2: track 35.3 -> 33.6 mm
- net CFG3: track 37.5 -> 38.1 mm
Other:
- board text added: "JLCJLCJLCJLC"
- board text removed: "JLCJLCJLC"

Commit message: fixed bom & updated prod files
Parts:
- J1: value USB_C_Receptacle -> 1054500101
- J6: value Screw_Terminal_01x02 -> 282834-2
- SW1: value SW_DIP_x03 -> DS04-254-1L-03BK
- U2, U3: value LM317_SOT-223 -> LM317DCYR
